File: Placa_Rediseñada/Placa_Rediseñada.kicad_sch (KiCad schematic)
At the start: 0 parts

Commit message: 好
Parts:
- added A1: Arduino_Nano_Every, Module:Arduino_Nano, symbol MCU_Module:Arduino_Nano_Every
- added BT1: Battery, Connector_PinSocket_2.54mm:PinSocket_1x03_P2.54mm_Vertical, symbol Device:Battery
- added BZ1: Buzzer, Buzzer_Beeper:Buzzer_12x9.5RM7.6, symbol Device:Buzzer
- added HL1, HR1: Conn_01x03_MountingPin, Connector_PinSocket_2.54mm:PinSocket_1x03_P2.54mm_Vertical, symbol Connector_Generic_MountingPin:Conn_01x03_MountingPin
- added J2: LineSensor, Connector_PinHeader_2.54mm:PinHeader_1x11_P2.54mm_Vertical, symbol Connector_Generic_MountingPin:Conn_01x11_MountingPin
- added J3, J5: Conn_01x08, Connector_PinHeader_2.54mm:PinHeader_1x08_P2.54mm_Vertical, symbol Connector_Generic:Conn_01x08
- added ML1, MR1, Motor1: Motor_DC, Connector_PinHeader_2.54mm:PinHeader_1x02_P2.54mm_Vertical, symbol Motor:Motor_DC
- added R1: 47KΩ, Resistor_THT:R_Axial_DIN0204_L3.6mm_D1.6mm_P7.62mm_Horizontal, symbol Device:R
- added R2, R3: 10KΩ, Resistor_THT:R_Axial_DIN0204_L3.6mm_D1.6mm_P7.62mm_Horizontal, symbol Device:R
- added SW1: SW_Nidec_CAS-120A1, Button_Switch_THT:SW_Slide-03_Wuerth-WS-SLTV_10x2.5x6.4_P2.54mm, symbol Switch:SW_Nidec_CAS-120A1
- added SW2, SW3, SW4: SW_Push, Button_Switch_THT:SW_PUSH_6mm_H5mm, symbol Switch:SW_Push
Connections:
- new net: BT1.1 (+), SW1.2 (B)
- new net 7.4V: A1.30 (VIN), J3.1 (Pin_1), SW1.3 (A)
- new net A01: J3.4 (Pin_4), ML1.1 (+)
- new net A02: J3.5 (Pin_5), ML1.2 (-)
- new net AIN1: A1.7 (D4), J5.2 (Pin_2)
- new net AIN2: A1.8 (D5), J5.3 (Pin_3)
- new net B01: J3.7 (Pin_7), MR1.1 (+)
- new net B02: J3.6 (Pin_6), MR1.2 (-)
- new net BIN1: A1.9 (D6), J5.5 (Pin_5)
- new net BIN2: A1.10 (D7), J5.6 (Pin_6)
- new net BUTTON: A1.12 (D9), R1.2, SW2.2
- new net BUZZER: A1.13 (D10), BZ1.1 (+)
- new net D1: A1.20 (A1), J2.4 (Pin_4)
- new net D2: A1.21 (A2), J2.5 (Pin_5)
- new net D3: A1.22 (A3), J2.6 (Pin_6)
- new net D4: A1.23 (SDA/A4), J2.7 (Pin_7)
- new net D5: A1.24 (SCL/A5), J2.8 (Pin_8)
- new net D6: A1.25 (A6), J2.9 (Pin_9)
- new net GND: A1.29 (GND), A1.4 (GND), BT1.2 (-), BZ1.2 (-), HL1.3 (Pin_3), HR1.3 (Pin_3), J2.1 (Pin_1), J3.3 (Pin_3), J3.8 (Pin_8), J5.8 (Pin_8), Motor1.2 (-), R1.1, R2.1, R3.1
- new net HL: A1.26 (A7), A1.28 (~{RESET}), HL1.1 (Pin_1)
- new net HR: A1.19 (A0), HR1.1 (Pin_1)
- new net LEDON: A1.14 (MOSI), J2.2 (Pin_2)
- new net PWMA: A1.6 (D3), J5.1 (Pin_1)
- new net PWMB: A1.11 (D8), J5.7 (Pin_7)
- new net Pin3: Motor1.1 (+)
- new net VCC: A1.27 (+5V), HL1.2 (Pin_2), HR1.2 (Pin_2), J2.11 (Pin_11), J3.2 (Pin_2), J5.4 (Pin_4), SW2.1, SW3.1, SW4.1
- new net 电钮1: A1.5 (D2), R2.2, SW4.2
- new net 电钮2: A1.15 (MISO), R3.2, SW3.2
- no-connect marks 0 -> 13
