File: Placa_Rediseñada/Placa_Rediseñada.kicad_pcb (KiCad board)
At the start: 2 copper layers, 100 x 100 mm, 31 parts, among them J2 LineSensor, J3 Conn_01x08, J5 Conn_01x08, SW1 SW_Nidec_CAS-120A1, SW2 SW_Push, SW3 SW_Push, SW4 SW_Push

Commit message: 牛肉
Parts:
- Motor A: renamed from ML1
- Motor B: renamed from MR1
- moved G*** 45.6 mm to (203.1, 93.9)
- moved BT1 15.2 mm to (116.8, 114.4)
- moved BZ1 14.8 mm to (170.9, 113.6)
- moved SW1 8.11 mm to (122.5, 96.7)
- renumbered SW2 to BUTTON, J2 to GND, HL1 to HL, SW4 to 电钮1, SW3 to 电钮2
Connections:
- REF** pad 1: (no net) -> LEDON (x2)
- REF** pad 1: (no net) -> VCC (x2)
- REF** pad 1: (no net) -> 电钮1 (x2)
Routing:
- net BUZZER: track 27.0 -> 12.3 mm
- net VCC: track 269.4 -> 259.4 mm
- net Net-(BT1-+): track 22.7 -> 15.6 mm
- net HL: track 54.4 -> 57.3 mm
- added copper zone on F.Cu, net GND
Other:
- board size 100 x 100 mm -> 100 x 101.5 mm
- board text added: "GND"
- board text added: "HL"
- board text added: "HR"
- board text added: "LEDON"
- board text added: "VCC"
- board text added: "电钮1"
